File: dispatcher.sch (KiCad schematic (older format))
At the start: 9 parts, among them P4 CONN_01X02, P5 CONN_01X02, P6 CONN_01X02, SW2 SW_PUSH, SW3 SW_PUSH

Commit message: release1
Parts:
- added D6, D7: LED, LEDs:LED-3MM, symbol LED
- added P7, P8: CONN_01X02, Connect:AK300-2, symbol CONN_01X02
- added R11, R12: R, Discret:R3-5, symbol R
- added SW4, SW5: SW_PUSH, Buttons_Switches_ThroughHole:SW_PUSH_SMALL, symbol SW_PUSH
Connections:
- net GND: now also D6.1 (K), D7.1 (K)
- net VCC: now also SW4.1, SW5.1
- new net: D6.2 (A), R11.1
- new net: D7.2 (A), R12.1
- new net IND_3: P7.1 (P1), R11.2
- new net IND_4: P8.1 (P1), R12.2
- new net SWI_3: P7.2 (P2), SW4.2
- new net SWI_4: P8.2 (P2), SW5.2
Changed lines of the file:
@@
 $EndComp
 $Comp
-L VCC #PWR06
+L VCC #PWR3
 U 1 1 569C7F94
 P 1350 1200
-F 0 "#PWR06" H 1350 1050 50  0001 C CNN
+F 0 "#PWR3" H 1350 1050 50  0001 C CNN
 F 1 "VCC" H 1350 1350 50  0000 C CNN
 F 2 "" H 1350 1200 50  0000 C CNN
@@
 $EndComp
 $Comp
-L GND #PWR07
+L GND #PWR4
 U 1 1 569C7FC8
 P 2050 1550
-F 0 "#PWR07" H 2050 1300 50  0001 C CNN
+F 0 "#PWR4" H 2050 1300 50  0001 C CNN
 F 1 "GND" H 2050 1400 50  0000 C CNN
 F 2 "" H 2050 1550 50  0000 C CNN
@@
 $EndComp
 $Comp
-L PWR_FLAG #FLG08
+L PWR_FLAG #FLG4
 U 1 1 569C8018
 P 1350 1750
-F 0 "#FLG08" H 1350 1845 50  0001 C CNN
+F 0 "#FLG4" H 1350 1845 50  0001 C CNN
 F 1 "PWR_FLAG" H 1350 1930 50  0000 C CNN
 F 2 "" H 1350 1750 50  0000 C CNN
@@
 $EndComp
 $Comp
-L PWR_FLAG #FLG09
+L PWR_FLAG #FLG5
 U 1 1 569C8052
 P 2300 950
-F 0 "#FLG09" H 2300 1045 50  0001 C CNN
+F 0 "#FLG5" H 2300 1045 50  0001 C CNN
 F 1 "PWR_FLAG" H 2300 1130 50  0000 C CNN
 F 2 "" H 2300 950 50  0000 C CNN
@@
 	0    -1   -1   0
 $EndComp
-Connection ~ 1800 1200
-Wire Wire Line
-	2300 1200 1800 1200
-Wire Wire Line
-	2300 950  2300 1200
-Connection ~ 1700 1900
-Wire Wire Line
-	1700 1900 1350 1900
-Wire Wire Line
-	1350 1900 1350 1750
-Connection ~ 1800 1400
-Wire Wire Line
-	2050 1400 2050 1550
-Wire Wire Line
-	1800 1400 2050 1400
-Connection ~ 1700 1400
-Wire Wire Line
-	1350 1400 1700 1400
-Wire Wire Line
-	1350 1200 1350 1400
-Wire Wire Line
-	1800 1100 1800 3450
-Wire Wire Line
-	1700 1100 1700 3100
-Wire Wire Line
-	2900 2500 2750 2500
-Wire Wire Line
-	1800 2500 2350 2500
-Wire Wire Line
-	3000 2150 3400 2150
-Wire Wire Line
-	1700 2150 2400 2150
 $Comp
 L SW_PUSH SW3
@@
 	0    -1   -1   0
 $EndComp
-Wire Wire Line
-	2900 3450 2750 3450
-Wire Wire Line
-	3000 3100 4300 3100
 Text GLabel 2850 1800 0    60   Input ~ 0
 SWI_1
-Wire Wire Line
-	2850 1800 3400 1800
 Text GLabel 3850 1800 0    60   Input ~ 0
 SWI_2
 Text GLabel 3750 2100 2    60   Input ~ 0
 IND_1
-Text GLabel 4750 2100 2    60   Input ~ 0
+Text GLabel 4500 2100 2    60   Input ~ 0
 IND_2
+$Comp
+L SW_PUSH SW4
+U 1 1 569CBEF0
+P 2700 4050
+F 0 "SW4" H 2850 4160 50  0000 C CNN
+F 1 "SW_PUSH" H 2700 3970 50  0000 C CNN
+F 2 "Buttons_Switches_ThroughHole:SW_PUSH_SMALL" H 2700 4050 50  0001 C CNN
+F 3 "" H 2700 4050 50  0000 C CNN
+	1    2700 4050
+	1    0    0    -1
+$EndComp
+$Comp
+L LED D6
+U 1 1 569CBEF6
+P 2550 4400
+F 0 "D6" H 2550 4500 50  0000 C CNN
+F 1 "LED" H 2550 4300 50  0000 C CNN
+F 2 "LEDs:LED-3MM" H 2550 4400 50  0001 C CNN
+F 3 "" H 2550 4400 50  0000 C CNN
+	1    2550 4400
+	1    0    0    -1
+$EndComp
+$Comp
+L R R11
+U 1 1 569CBEFC
+P 3050 4400
+F 0 "R11" V 3130 4400 50  0000 C CNN
+F 1 "R" V 3050 4400 50  0000 C CNN
+F 2 "Discret:R3-5" V 2980 4400 50  0001 C CNN
+F 3 "" H 3050 4400 50  0000 C CNN
+	1    3050 4400
+	0    -1   -1   0
+$EndComp
+$Comp
+L SW_PUSH SW5
+U 1 1 569CC2DE
+P 2700 5050
+F 0 "SW5" H 2850 5160 50  0000 C CNN
+F 1 "SW_PUSH" H 2700 4970 50  0000 C CNN
+F 2 "Buttons_Switches_ThroughHole:SW_PUSH_SMALL" H 2700 5050 50  0001 C CNN
+F 3 "" H 2700 5050 50  0000 C CNN
+	1    2700 5050
+	1    0    0    -1
+$EndComp
+$Comp
+L LED D7
+U 1 1 569CC2E4
+P 2550 5400
+F 0 "D7" H 2550 5500 50  0000 C CNN
+F 1 "LED" H 2550 5300 50  0000 C CNN
+F 2 "LEDs:LED-3MM" H 2550 5400 50  0001 C CNN
+F 3 "" H 2550 5400 50  0000 C CNN
+	1    2550 5400
+	1    0    0    -1
+$EndComp
+$Comp
+L R R12
+U 1 1 569CC2EA
+P 3050 5400
+F 0 "R12" V 3130 5400 50  0000 C CNN
+F 1 "R" V 3050 5400 50  0000 C CNN
+F 2 "Discret:R3-5" V 2980 5400 50  0001 C CNN
+F 3 "" H 3050 5400 50  0000 C CNN
+	1    3050 5400
+	0    -1   -1   0
+$EndComp
+$Comp
+L CONN_01X02 P7
+U 1 1 569CC4C6
+P 5350 1500
+F 0 "P7" H 5350 1650 50  0000 C CNN
+F 1 "CONN_01X02" V 5450 1500 50  0000 C CNN
+F 2 "Connect:AK300-2" H 5350 1500 50  0001 C CNN
+F 3 "" H 5350 1500 50  0000 C CNN
+	1    5350 1500
+	0    -1   -1   0
+$EndComp
+$Comp
+L CONN_01X02 P8
+U 1 1 569CC606
+P 6300 1500
+F 0 "P8" H 6300 1650 50  0000 C CNN
+F 1 "CONN_01X02" V 6400 1500 50  0000 C CNN
+F 2 "Connect:AK300-2" H 6300 1500 50  0001 C CNN
+F 3 "" H 6300 1500 50  0000 C CNN
+	1    6300 1500
+	0    -1   -1   0
+$EndComp
+Connection ~ 1800 1200
+Wire Wire Line
+	2300 1200 1800 1200
+Wire Wire Line
+	2300 950  2300 1200
+Connection ~ 1700 1900
+Wire Wire Line
+	1700 1900 1350 1900
+Wire Wire Line
+	1350 1900 1350 1750
+Connection ~ 1800 1400
+Wire Wire Line
+	2050 1400 2050 1550
+Wire Wire Line
+	1800 1400 2050 1400
+Connection ~ 1700 1400
+Wire Wire Line
+	1350 1400 1700 1400
+Wire Wire Line
+	1350 1200 1350 1400
+Wire Wire Line
+	1800 1100 1800 5400
+Wire Wire Line
+	1700 1100 1700 5050
+Wire Wire Line
+	2900 2500 2750 2500
+Wire Wire Line
+	1800 2500 2350 2500
+Wire Wire Line
+	3000 2150 3400 2150
+Wire Wire Line
+	1700 2150 2400 2150
+Wire Wire Line
+	2900 3450 2750 3450
+Wire Wire Line
+	3000 3100 4300 3100
+Wire Wire Line
+	2850 1800 3400 1800
 Connection ~ 1800 2500
 Connection ~ 1700 2150
@@
 	3850 1800 4300 1800
 Connection ~ 4300 1800
-Wire Wire Line
-	4750 2100 4200 2100
 Connection ~ 4200 2100
 Wire Wire Line
@@
 Wire Wire Line
 	4200 3450 4200 1700
+Wire Wire Line
+	4200 2100 4500 2100
+Wire Wire Line
+	2900 4400 2750 4400
+Wire Wire Line
+	5400 4050 3000 4050
+Wire Wire Line
+	1700 4050 2400 4050
+Wire Wire Line
+	1800 4400 2350 4400
+Wire Wire Line
+	5300 4400 3200 4400
+Wire Wire Line
+	2900 5400 2750 5400
+Wire Wire Line
+	6350 5050 3000 5050
+Wire Wire Line
+	1700 5050 2400 5050
+Wire Wire Line
+	1800 5400 2350 5400
+Wire Wire Line
+	6250 5400 3200 5400
+Connection ~ 1800 3450
+Connection ~ 1800 4400
+Connection ~ 1700 3100
+Connection ~ 1700 4050
+Connection ~ 5400 1800
+Connection ~ 5300 2100
+Wire Wire Line
+	5400 1700 5400 4050
+Wire Wire Line
+	5300 1700 5300 4400
+Connection ~ 6350 1800
+Connection ~ 6250 2100
+Wire Wire Line
+	6350 1700 6350 5050
+Wire Wire Line
+	6250 1700 6250 5400
+Text GLabel 4950 1800 0    60   Input ~ 0
+SWI_3
+Text GLabel 6000 1800 0    60   Input ~ 0
+SWI_4
+Text GLabel 5650 2100 2    60   Input ~ 0
+IND_3
+Text GLabel 6600 2100 2    60   Input ~ 0
+IND_4
+Wire Wire Line
+	5300 2100 5650 2100
+Wire Wire Line
+	6250 2100 6600 2100
+Wire Wire Line
+	6350 1800 6000 1800
+Wire Wire Line
+	5400 1800 4950 1800
 $EndSCHEMATC
