File: pointkey.kicad_pcb (KiCad board)
At the start: 2 copper layers, 12 parts, among them P1 CONN_01X02, SW1 SW_PUSH, SW2 SW_PUSH, U1 4013

Commit message: new pcb
Parts:
- removed D3: LED, LEDs:LED-3MM
- removed SW2: SW_PUSH, Buttons_Switches_ThroughHole:SW_PUSH_SMALL
- added D1: D, Discret:D4, F.Cu at (69.6, 38.6)
- added K1: RELAY_1RT, kicad_my_library:RELAY_812H_1C_C, F.Cu at (95.2, 32.9)
- added P2: CONN_01X03, Pin_Headers:Pin_Header_Straight_1x03, F.Cu at (96.1, 43.4)
- added Q1: КТ315, kicad_my_library:кт-13, F.Cu at (78.9, 28.7)
- C1: value C -> 1u
- C2: value C -> 20u
- D2: value LED -> D; footprint LEDs:LED-3MM -> Discret:D4
- R1, R3: value R -> 22k
- R2: value R -> 510k
- R4: value R -> 10k
- moved SW1 159.8 mm to (31.4, 34.4)
- moved R3 116.3 mm to (57.8, 32.9), turned to 90 degrees
- moved D2 112.8 mm to (74.8, 33.8), turned to 270 degrees
- moved U1 111.2 mm to (48.3, 42.4), turned to 180 degrees
- moved R4 103.8 mm to (80.6, 39.6), turned to 270 degrees
- moved R2 95.3 mm to (63.9, 39.2), turned to 270 degrees
- moved R1 95.1 mm to (53.0, 32.9), turned to 270 degrees
- moved C2 89.1 mm to (57.7, 42.2), turned to 180 degrees
- moved C1 85.4 mm to (63.9, 28.6), turned to 90 degrees
- moved P1 84.4 mm to (91.8, 43.6), turned to 270 degrees
Connections:
- C2 pad 1: Net-(C2-Pad1) -> VCC
- C2 pad 2: GND -> Net-(C2-Pad2)
- D2 pad 1: GND -> VCC
- R1 pad 1: Net-(C1-Pad1) -> Net-(R1-Pad1)
- R2 pad 1: Net-(C2-Pad1) -> Net-(C1-Pad1)
- R2 pad 2: GND -> Net-(D1-Pad1)
- R3 pad 1: Net-(D2-Pad2) -> Net-(C2-Pad2)
- R3 pad 2: Net-(R3-Pad2) -> GND
- SW1 pad 1: Net-(C1-Pad1) -> Net-(R1-Pad1)
- U1 pad 1: Net-(R3-Pad2) -> Net-(D1-Pad1)
- U1 pad 10: GND -> Net-(C2-Pad2)
- U1 pad 11: Net-(C2-Pad1) -> Net-(D1-Pad1)
- U1 pad 3: Net-(C1-Pad1) -> GND
- U1 pad 4: GND -> Net-(C1-Pad1)
- U1 pad 5: Net-(U1-Pad2) -> GND
- U1 pad 6: GND -> Net-(R1-Pad1)
Routing:
- net Net-(C2-Pad1): track 90.0 -> 0.00 mm
- net GND: track 177.0 -> 105.4 mm
- net Net-(C1-Pad1): track 98.6 -> 28.1 mm
- net VCC: track 56.6 -> 107.2 mm
- net Net-(R1-Pad1): track 0.00 -> 37.9 mm
- net Net-(D1-Pad1): track 0.00 -> 36.5 mm
- net Net-(R4-Pad2): track 14.7 -> 44.1 mm
- net Net-(K1-Pad5): track 0.00 -> 17.6 mm
- net Net-(K1-Pad3): track 0.00 -> 17.1 mm
- net Net-(U1-Pad2): track 12.2 -> 0.00 mm
- net Net-(R3-Pad2): track 9.79 -> 0.00 mm
- net Net-(D2-Pad2): track 6.52 -> 15.2 mm
- net Net-(C2-Pad2): track 0.00 -> 5.91 mm
- net Net-(K1-Pad4): track 0.00 -> 4.55 mm
- net Net-(Q1-Pad2): track 8.01 -> 3.99 mm
Other:
- net class big added: clearance 0.7, trace_width 1, via_dia 0.5, via_drill 0.4

Commit message: fixes
Parts:
- moved SW1 10.8 mm to (22.2, 28.8)
- moved C1 8.27 mm to (57.8, 23.0)
- moved C2 8.27 mm to (51.6, 36.6)
- moved K1 8.27 mm to (89.2, 27.3)
- moved Q1 8.27 mm to (72.8, 23.1)
- moved R1 8.27 mm to (46.9, 27.3)
- moved R2 8.27 mm to (57.8, 33.7)
- moved D1 8.27 mm to (63.5, 33.0)
- moved D2 8.27 mm to (68.7, 28.2)
- moved R3 8.27 mm to (51.7, 27.3)
- moved U1 8.27 mm to (42.2, 36.8)
- moved R4 8.27 mm to (74.5, 34.0)
- moved P1 6.56 mm to (85.7, 41.1)
- moved P2 6.49 mm to (90.0, 41.2)
Routing:
- net Net-(C2-Pad2): track 5.91 -> 52.7 mm, vias 0 -> 2
- net VCC: track 107.2 -> 111.2 mm
- net Net-(K1-Pad3): track 17.1 -> 20.5 mm
- net Net-(K1-Pad5): track 17.6 -> 21.0 mm
- net Net-(K1-Pad4): track 4.55 -> 7.92 mm
- net GND: track 105.4 -> 108.6 mm
- net Net-(R1-Pad1): track 37.9 -> 39.3 mm
- added copper zone on B.Cu, net (none)

Commit message: transistor key for indicator led
Parts:
- added D3: LED, LEDs:LED-3MM, F.Cu at (78.0, 14.9)
- added Q2: КТ315, kicad_my_library:кт-13, F.Cu at (73.1, 9.33)
- added R5: 2,2K, Discret:R3-5, F.Cu at (104.1, 20.4)
Changed lines of the file:
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@@
 (kicad_pcb (version 4) (host pcbnew 4.0.1-3.201512221402+6198~38~ubuntu14.04.1-stable)
   (general
-    (links 33)
-    (no_connects 0)
-    (area 12.065 11.8745 104.775001 49.276001)
+    (links 38)
+    (no_connects 5)
+    (area 0 0 0 0)
     (thickness 1.6)
     (drawings 0)
     (tracks 111)
     (zones 0)
-    (modules 14)
-    (nets 15)
+    (modules 17)
+    (nets 17)
   )
   (page A4)
@@
   (net 13 "Net-(Q1-Pad2)")
   (net 14 "Net-(R1-Pad1)")
+  (net 15 "Net-(D3-Pad1)")
+  (net 16 "Net-(Q2-Pad2)")
   (net_class Default "This is the default net class."
     (clearance 0.7)
@@
     (add_net "Net-(D1-Pad1)")
     (add_net "Net-(D2-Pad2)")
+    (add_net "Net-(D3-Pad1)")
     (add_net "Net-(K1-Pad3)")
     (add_net "Net-(K1-Pad4)")
     (add_net "Net-(K1-Pad5)")
     (add_net "Net-(Q1-Pad2)")
+    (add_net "Net-(Q2-Pad2)")
     (add_net "Net-(R1-Pad1)")
     (add_net "Net-(R4-Pad2)")
@@
       (rotate (xyz 0 0 0))
     )
+  )
+  (module LEDs:LED-3MM (layer F.Cu)
+    (at 77.978 14.859)
+    (descr "LED 3mm round vertical")
+    (tags "LED  3mm round vertical")
+    (fp_text reference D3 (at 1.91 3.06) (layer F.SilkS)
+      (effects (font (size 1 1) (thickness 0.15)))
+    )
+    (fp_text value LED (at 1.3 -2.9) (layer F.Fab)
+      (effects (font (size 1 1) (thickness 0.15)))
+    )
+    (fp_line (start -1.2 2.3) (end 3.8 2.3) (layer F.CrtYd) (width 0.05))
+    (fp_line (start 3.8 2.3) (end 3.8 -2.2) (layer F.CrtYd) (width 0.05))
+    (fp_line (start 3.8 -2.2) (end -1.2 -2.2) (layer F.CrtYd) (width 0.05))
+    (fp_line (start -1.2 -2.2) (end -1.2 2.3) (layer F.CrtYd) (width 0.05))
+    (fp_line (start -0.199 1.314) (end -0.199 1.114) (layer F.SilkS) (width 0.15))
+    (fp_line (start -0.199 -1.28) (end -0.199 -1.1) (layer F.SilkS) (width 0.15))
+    (fp_arc (start 1.301 0.034) (end -0.199 -1.286) (angle 108.5) (layer F.SilkS) (width 0.15))
+    (fp_arc (start 1.301 0.034) (end 0.25 -1.1) (angle 85.7) (layer F.SilkS) (width 0.15))
+    (fp_arc (start 1.311 0.034) (end 3.051 0.994) (angle 110) (layer F.SilkS) (width 0.15))
+    (fp_arc (start 1.301 0.034) (end 2.335 1.094) (angle 87.5) (layer F.SilkS) (width 0.15))
+    (fp_text user K (at -1.69 1.74) (layer F.SilkS)
+      (effects (font (size 1 1) (thickness 0.15)))
+    )
+    (pad 1 thru_hole rect (at 0 0 90) (size 2 2) (drill 1.00076) (layers *.Cu *.Mask F.SilkS)
+      (net 15 "Net-(D3-Pad1)"))
+    (pad 2 thru_hole circle (at 2.54 0) (size 2 2) (drill 1.00076) (layers *.Cu *.Mask F.SilkS)
+      (net 7 VCC))
+    (model LEDs.3dshapes/LED-3MM.wrl
+      (at (xyz 0.05 0 0))
+      (scale (xyz 1 1 1))
+      (rotate (xyz 0 0 90))
+    )
+  )
+  (module Discret:R3-5 (layer F.Cu)
+    (at 104.0765 20.447 90)
+    (fp_text reference R5 (at 0 0 90) (layer F.SilkS)
+      (effects (font (size 1 1) (thickness 0.15)))
+    )
+    (fp_text value 2,2K (at 0 0 90) (layer F.Fab)
+      (effects (font (size 1 1) (thickness 0.15)))
+    )
+    (fp_line (start -3.81 -0.635) (end -3.81 1.27) (layer F.SilkS) (width 0.15))
+    (fp_line (start -3.81 1.27) (end 3.81 1.27) (layer F.SilkS) (width 0.15))
+    (fp_line (start 3.81 1.27) (end 3.81 -1.27) (layer F.SilkS) (width 0.15))
+    (fp_line (start 3.81 -1.27) (end -3.81 -1.27) (layer F.SilkS) (width 0.15))
+    (fp_line (start -3.81 -1.27) (end -3.81 -0.635) (layer F.SilkS) (width 0.15))
+    (fp_line (start -4.445 0) (end -3.81 0) (layer F.SilkS) (width 0.15))
+    (fp_line (start 3.81 0) (end 4.445 0) (layer F.SilkS) (width 0.15))
+    (fp_line (start -3.81 -0.635) (end -3.175 -1.27) (layer F.SilkS) (width 0.15))
+    (pad 1 thru_hole circle (at -4.445 0 90) (size 1.397 1.397) (drill 0.8128) (layers *.Cu *.Mask F.SilkS)
+      (net 5 "Net-(R4-Pad2)"))
+    (pad 2 thru_hole circle (at 4.445 0 90) (size 1.397 1.397) (drill 0.8128) (layers *.Cu *.Mask F.SilkS)
+      (net 16 "Net-(Q2-Pad2)"))
+    (model Discret.3dshapes/R3-5.wrl
+      (at (xyz 0 0 0))
+      (scale (xyz 0.35 0.35 0.3))
+      (rotate (xyz 0 0 0))
+    )
+  )
+  (module kicad_my_library:кт-13 (layer F.Cu)
+    (at 73.0885 9.3345)
+    (fp_text reference Q2 (at 0.25 1.25) (layer F.SilkS)
+      (effects (font (size 1 1) (thickness 0.15)))
+    )
+    (fp_text value КТ315 (at 0 -4.75) (layer F.Fab)
+      (effects (font (size 1 1) (thickness 0.15)))
+    )
+    (fp_line (start -3.5 -3) (end -3.5 0) (layer F.SilkS) (width 0.15))
+    (fp_line (start -3.5 0) (end 3.5 0) (layer F.SilkS) (width 0.15))
+    (fp_line (start 3.5 -3) (end -3.5 -3) (layer F.SilkS) (width 0.15))
+    (fp_line (start 3.5 -2.25) (end -3.5 -2.25) (layer F.SilkS) (width 0.15))
+    (fp_line (start 3.5 -3) (end 3.5 0) (layer F.SilkS) (width 0.15))
+    (pad 2 thru_hole oval (at 2.5 -1.75) (size 1.8 2.2) (drill 0.8) (layers *.Cu *.Mask F.SilkS)
+      (net 16 "Net-(Q2-Pad2)"))
+    (pad 3 thru_hole oval (at -2.5 -1.75) (size 1.8 2.2) (drill 0.8) (layers *.Cu *.Mask F.SilkS)
+      (net 6 GND))
+    (pad 1 thru_hole oval (at 0 -1.75) (size 1.8 2.2) (drill 0.8) (layers *.Cu *.Mask F.SilkS)
+      (net 15 "Net-(D3-Pad1)"))
   )
   (segment (start 57.785 29.21) (end 62.23 29.21) (width 0.7) (layer B.Cu) (net 1))
@@
   (segment (start 38.989 30.48) (end 38.989 26.67) (width 0.7) (layer B.Cu) (net 6))
   (segment (start 40.259 31.75) (end 38.989 30.48) (width 0.7) (layer B.Cu) (net 6))
-  (segment (start 34.544 36.83) (end 31.4325 36.83) (width 0.7) (layer B.Cu) (net 7) (status 400000))
-  (segment (start 31.4325 36.83) (end 25.9715 31.369) (width 0.7) (layer B.Cu) (net 7) (status 800000))
+  (segment (start 34.544 36.83) (end 31.4325 36.83) (width 0.7) (layer B.Cu) (net 7))
+  (segment (start 31.4325 36.83) (end 25.9715 31.369) (width 0.7) (layer B.Cu) (net 7))
   (segment (start 78.359 42.799) (end 81.534 42.799) (width 0.7) (layer B.Cu) (net 7))
   (segment (start 36.322 36.83) (end 42.291 42.799) (width 0.7) (layer B.Cu) (net 7))
@@
   (segment (start 74.521 25.614) (end 74.521 29.563) (width 0.7) (layer B.Cu) (net 13))
   (segment (start 74.521 29.563) (end 74.549 29.591) (width 0.7) (layer B.Cu) (net 13))
-  (segment (start 25.9715 26.289) (end 25.9715 26.2255) (width 0.7) (layer B.Cu) (net 14) (status C00000))
-  (segment (start 25.9715 26.2255) (end 33.401 18.796) (width 0.7) (layer B.Cu) (net 14) (status 400000))
+  (segment (start 25.9715 26.289) (end 25.9715 26.2255) (width 0.7) (layer B.Cu) (net 14))
+  (segment (start 25.9715 26.2255) (end 33.401 18.796) (width 0.7) (layer B.Cu) (net 14))
   (segment (start 46.863 21.844) (end 46.863 22.86) (width 0.7) (layer B.Cu) (net 14))
   (segment (start 43.815 18.796) (end 46.863 21.844) (width 0.7) (layer B.Cu) (net 14))

Commit message: dispatcher
Parts:
- added D4: LED, LEDs:LED-3MM, F.Cu at (50.5, 43.8)
- added D5: LED, LEDs:LED-3MM, F.Cu at (50.5, 28.2)
- added P3: CONN_01X02, Connect:AK300-2, F.Cu at (128.8, 43.8)
- added P4: CONN_01X02, Connect:AK300-2, F.Cu at (82.9, 58.6)
- added P5: CONN_01X02, Connect:AK300-2, F.Cu at (83.0, 43.8)
- added P6: CONN_01X02, Connect:AK300-2, F.Cu at (83.0, 28.2)
- added Q3: КТ315, kicad_my_library:кт-13, F.Cu at (215.2, 43.5)
- added Q4: КТ315, kicad_my_library:кт-13, F.Cu at (207.5, 59.5)
- added R10: R, Discret:R3-5, F.Cu at (66.0, 28.2)
- added R6: 100, Discret:R3-5, F.Cu at (199.0, 47.5)
- added R7: 1K, Discret:R3-5, F.Cu at (196.0, 41.8)
- added R8: 1k, Discret:R3-5, F.Cu at (194.5, 57.8)
- added R9: R, Discret:R3-5, F.Cu at (66.5, 43.8)
- added SW2: SW_PUSH, Buttons_Switches_ThroughHole:SW_PUSH_SMALL, F.Cu at (37.5, 43.8)
- added SW3: SW_PUSH, Buttons_Switches_ThroughHole:SW_PUSH_SMALL, F.Cu at (37.5, 28.2)
- D2: value D -> LED; footprint Discret:D4 -> LEDs:LED-3MM
- D3: value LED -> D; footprint LEDs:LED-3MM -> Discret:D4
- P1: footprint Pin_Headers:Pin_Header_Straight_1x02 -> Connect:AK300-2
- P2: value CONN_01X03 -> CONN_01X02; footprint Pin_Headers:Pin_Header_Straight_1x03 -> Connect:AK300-2
- R4: value 10k -> 100
- R5: value 2,2K -> 100
- moved P2 160.7 mm to (250.8, 37.5), turned to 270 degrees
- moved D2 159.5 mm to (225.2, 58.8), turned to 90 degrees
- moved K1 159.2 mm to (246.0, 54.5)
- moved D3 155.3 mm to (230.2, 45.5), turned to 90 degrees
- moved Q1 149.1 mm to (218.5, 54.5), turned to 90 degrees
- moved Q2 138.3 mm to (203.2, 56.0), turned to 90 degrees
- moved R3 135.8 mm to (184.0, 57.8), turned to 270 degrees
- moved R4 134.9 mm to (209.0, 45.0)
- moved C2 132.5 mm to (184.0, 41.8), turned to 90 degrees
- moved U1 128.1 mm to (170.0, 45.0), turned to 0 degrees
- moved SW1 126.2 mm to (144.8, 59.0), turned to 180 degrees
- moved R5 122.4 mm to (224.0, 45.0)
- moved R1 116.0 mm to (158.8, 57.8), turned to 180 degrees
- moved C1 107.4 mm to (161.0, 52.8)
- moved D1 90.3 mm to (152.5, 48.5), turned to 90 degrees
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Connections:
- net Net-(R1-Pad1) renamed SWI_1
- D2 pad 1: VCC -> Net-(D2-Pad1)
- D3 pad 1: Net-(D3-Pad1) -> VCC
- D3 pad 2: VCC -> Net-(D3-Pad2)
- K1 pad 1: Net-(D2-Pad2) -> VCC
- K1 pad 2: VCC -> Net-(D3-Pad2)
- Q1 pad 1: Net-(D2-Pad2) -> Net-(D2-Pad1)
- Q2 pad 1: Net-(D3-Pad1) -> Net-(Q2-Pad1)
- R4 pad 1: Net-(Q1-Pad2) -> Net-(R4-Pad1)
- R4 pad 2: Net-(R4-Pad2) -> Net-(Q1-Pad2)
- R5 pad 1: Net-(R4-Pad2) -> Net-(D2-Pad2)
- R5 pad 2: Net-(Q2-Pad2) -> VCC
- U1 pad 13: Net-(R4-Pad2) -> Net-(R4-Pad1)
Routing:
- net VCC: track 111.2 -> 312.0 mm
- net GND: track 108.6 -> 266.5 mm
- net IND_1: track 0.00 -> 155.0 mm
- net SWI_1: track 39.3 -> 175.8 mm
- net SWI_2: track 0.00 -> 50.3 mm
- net Net-(R4-Pad1): track 0.00 -> 45.4 mm
- net Net-(D3-Pad2): track 0.00 -> 44.3 mm
- net Net-(R4-Pad2): track 44.1 -> 0.00 mm
- net Net-(Q2-Pad1): track 0.00 -> 36.5 mm
- net Net-(C2-Pad2): track 52.7 -> 29.7 mm
- net Net-(U1-Pad12): track 12.5 -> 31.8 mm
- net Net-(Q4-Pad2): track 0.00 -> 14.8 mm
- net Net-(K1-Pad5): track 21.0 -> 6.52 mm
- net IND_2: track 0.00 -> 12.6 mm
- net Net-(D2-Pad1): track 0.00 -> 11.1 mm
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Other:
- net class Default: clearance 0.7 -> 0.8; trace_width 0.7 -> 0.6
- net class big removed
- rule trace_clearance: 0.7 -> 0.8

Commit message: release1
Parts:
- added D6: LED, LEDs:LED-3MM, F.Cu at (59.8, 100.5)
- added D7: LED, LEDs:LED-3MM, F.Cu at (59.8, 85.2)
- added P7: CONN_01X02, Connect:AK300-2, F.Cu at (92.2, 100.5)
- added P8: CONN_01X02, Connect:AK300-2, F.Cu at (92.2, 85.2)
- added R11: R, Discret:R3-5, F.Cu at (75.2, 100.5)
- added R12: R, Discret:R3-5, F.Cu at (75.2, 85.2)
- added SW4: SW_PUSH, Buttons_Switches_ThroughHole:SW_PUSH_SMALL, F.Cu at (46.8, 100.5)
- added SW5: SW_PUSH, Buttons_Switches_ThroughHole:SW_PUSH_SMALL, F.Cu at (46.8, 85.2)
- moved C1 88.0 mm to (170.2, 140.2)
- moved C2 88.0 mm to (193.2, 129.2)
- moved D1 88.0 mm to (161.8, 136.0)
- moved D2 88.0 mm to (234.5, 146.2)
- moved D3 88.0 mm to (239.5, 133.0)
- moved D4 88.0 mm to (59.8, 131.2)
- moved D5 88.0 mm to (59.8, 115.8)
- moved K1 88.0 mm to (255.2, 142.0)
- moved P1 88.0 mm to (138.0, 141.2)
- moved P2 88.0 mm to (260.0, 125.0)
- moved P3 88.0 mm to (138.0, 131.2)
- moved P4 88.0 mm to (92.1, 146.1)
- moved P5 88.0 mm to (92.2, 131.2)
- moved P6 88.0 mm to (92.2, 115.8)
- moved Q1 88.0 mm to (227.8, 142.0)
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Routing:
- net GND: track 266.5 -> 368.4 mm
- net VCC: track 312.0 -> 374.6 mm
- net SWI_4: track 0.00 -> 50.3 mm
- net SWI_3: track 0.00 -> 50.3 mm
- net IND_4: track 0.00 -> 12.6 mm
- net IND_3: track 0.00 -> 12.6 mm
- net Net-(D7-Pad2): track 0.00 -> 8.52 mm
- net Net-(D6-Pad2): track 0.00 -> 8.52 mm
